File: bluekeeb-kicad/_autosave-bluekeeb.kicad_pcb (KiCad board)
At the start: 2 copper layers, 251 x 122.9 mm, 139 parts, among them SW1 SW_Push, SW10 SW_Push, SW11 SW_Push, SW12 SW_Push, SW13 SW_Push, SW14 SW_Push, SW15 SW_Push, SW16 SW_Push, SW17 SW_Push, SW18 SW_Push, SW19 SW_Push, SW2 SW_Push, SW20 SW_Push, SW21 SW_Push, SW22 SW_Push, SW23 SW_Push, SW24 SW_Push, SW25 SW_Push, SW26 SW_Push, SW27 SW_Push, SW28 SW_Push, SW29 SW_Push, SW3 SW_Push, SW30 SW_Push, SW31 SW_Push, SW32 SW_Push, SW33 SW_Push, SW34 SW_Push, SW35 SW_Push, SW36 SW_Push, SW37 SW_Push, SW38 SW_Push, SW39 SW_Push, SW4 SW_Push, SW40 SW_Push, SW41 SW_Push, SW42 SW_Push, SW43 SW_Push, SW44 SW_Push, SW45 SW_Push, SW46 SW_Push, SW47 SW_Push, SW48 SW_Push, SW49 SW_Push, SW5 SW_Push, SW50 SW_Push, SW51 SW_Push, SW52 SW_Push, SW53 SW_Push, SW54 SW_Push, SW55 SW_Push, SW56 SW_Push, SW57 SW_Push, SW58 SW_Push, SW59 SW_Push, SW6 SW_Push, SW60 SW_Push, SW7 SW_Push, SW8 SW_Push, SW9 SW_Push, U1 XIAO-nRF52840-SMD, U2 XIAO-nRF52840-SMD

Commit message: Finalllyyy i fixed my mousebites problem
Parts:
- removed H10, H11, H12, H13, H2, H4, H6, H7, H8, H9: MountingHole, panelization:mouse-bite-5mm-slot
- added SW61: RotaryEncoder, Rotary_Encoder:RotaryEncoder_Alps_EC11E-Switch_Vertical_H20mm, F.Cu at (61.8, 21.3)
- added SW62: RotaryEncoder, Rotary_Encoder:RotaryEncoder_Alps_EC11E-Switch_Vertical_H20mm, F.Cu at (230.9, 21.3)
Connections:
- U1 pad 17: unconnected-(U1-NFC1-Pad17) -> Net-(U1-NFC1)
- U1 pad 18: unconnected-(U1-NFC2-Pad18) -> Net-(U1-NFC2)
- U1 pad 22: unconnected-(U1-GND-Pad22) -> Net-(SW61-PadC)
- U2 pad 17: unconnected-(U2-NFC1-Pad17) -> Net-(U2-NFC1)
- U2 pad 18: unconnected-(U2-NFC2-Pad18) -> Net-(U2-NFC2)
- U2 pad 22: unconnected-(U2-GND-Pad22) -> Net-(SW62-PadC)
Routing:
- net Net-(U1-NFC1): track 0.00 -> 82.9 mm, vias 0 -> 2
- net Net-(U1-NFC2): track 0.00 -> 71.5 mm, vias 0 -> 2
- net Net-(U2-NFC1): track 0.00 -> 53.3 mm, vias 0 -> 1
- net Net-(U2-NFC2): track 0.00 -> 47.6 mm, vias 0 -> 1
- net Net-(SW62-PadC): track 0.00 -> 36.6 mm, vias 0 -> 1
- net Net-(D12-A): track 0.00 -> 23.8 mm, vias 0 -> 1
- net Net-(SW61-PadC): track 0.00 -> 18.3 mm, vias 0 -> 2
- net /left/col1: track 128.3 -> 131.0 mm
Other:
- board size 251 x 122.9 mm -> 253 x 126.5 mm
