File: bluekeeb-kicad/bluekeeb.kicad_pcb (KiCad board)
At the start: 2 copper layers, 251 x 122.9 mm, 139 parts, among them SW1 SW_Push, SW10 SW_Push, SW11 SW_Push, SW12 SW_Push, SW13 SW_Push, SW14 SW_Push, SW15 SW_Push, SW16 SW_Push, SW17 SW_Push, SW18 SW_Push, SW19 SW_Push, SW2 SW_Push, SW20 SW_Push, SW21 SW_Push, SW22 SW_Push, SW23 SW_Push, SW24 SW_Push, SW25 SW_Push, SW26 SW_Push, SW27 SW_Push, SW28 SW_Push, SW29 SW_Push, SW3 SW_Push, SW30 SW_Push, SW31 SW_Push, SW32 SW_Push, SW33 SW_Push, SW34 SW_Push, SW35 SW_Push, SW36 SW_Push, SW37 SW_Push, SW38 SW_Push, SW39 SW_Push, SW4 SW_Push, SW40 SW_Push, SW41 SW_Push, SW42 SW_Push, SW43 SW_Push, SW44 SW_Push, SW45 SW_Push, SW46 SW_Push, SW47 SW_Push, SW48 SW_Push, SW49 SW_Push, SW5 SW_Push, SW50 SW_Push, SW51 SW_Push, SW52 SW_Push, SW53 SW_Push, SW54 SW_Push, SW55 SW_Push, SW56 SW_Push, SW57 SW_Push, SW58 SW_Push, SW59 SW_Push, SW6 SW_Push, SW60 SW_Push, SW7 SW_Push, SW8 SW_Push, SW9 SW_Push, U1 XIAO-nRF52840-SMD, U2 XIAO-nRF52840-SMD

Commit message: Found an issue with pcb placement, started fixing
i had an error with windows 11 and unix file endings, and couldn't figure out how to make a git repo until not too long ago, so that's why my initial commit has a lot of stuff on it.
Parts:
- moved D54 197.6 mm to (255.7, 65.0)
- moved SW12 197.6 mm to (261.9, 50.0)
- moved SW54 197.6 mm to (261.9, 69.1)
- moved D8 189.0 mm to (217.6, 41.1)
- moved SW8 189.0 mm to (223.8, 45.2)
- moved D10 187.5 mm to (237.1, 45.9)
- moved SW10 187.5 mm to (242.9, 50.0)
- moved D44 186.1 mm to (218.1, 117.4)
- moved SW44 186.1 mm to (223.8, 121.4)
- moved SW51 158.7 mm to (121.4, 123.8)
- moved D30 155.5 mm to (199.0, 55.3)
- moved SW30 155.5 mm to (204.8, 59.5)
- moved D41 148.3 mm to (96.0, 93.6)
- moved SW41 148.3 mm to (102.4, 97.6)
- moved SW31 145.6 mm to (83.3, 83.3)
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Routing:
- net /left/col1: track 39.1 -> 0.00 mm
- net /left/col4: track 23.9 -> 55.1 mm
- net /right/col5: track 222.4 -> 230.3 mm

Commit message: save before plugin
Parts:
- moved TP1 242.0 mm to (33.0, 44.5)
- moved TP3 242.0 mm to (33.0, 51.0)
- moved TP2 241.6 mm to (275.0, 41.0)
- moved TP4 241.6 mm to (275.0, 48.5)
- moved U2 219.4 mm to (264.5, 28.5)
- moved U1 217.7 mm to (44.5, 28.5)
- moved D12 209.9 mm to (255.5, 45.0)
- moved D51 158.6 mm to (115.5, 119.0)
- moved D60 140.5 mm to (256.0, 121.5)
- moved D52 126.1 mm to (237.0, 121.5)
- moved D2 122.0 mm to (160.5, 47.5)
- moved D4 110.2 mm to (179.5, 42.6)
- moved D59 102.5 mm to (134.5, 123.5)
- moved D1 101.3 mm to (39.0, 45.0)
- moved D11 45.1 mm to (134.5, 47.5)
Routing:
- net /right/col3: track 356.8 -> 0.00 mm
- net /left/row3: track 232.8 -> 0.00 mm
- net /right/col5: track 230.3 -> 0.00 mm, vias 1 -> 0
- net /left/col5: track 144.4 -> 0.00 mm, vias 2 -> 0
- net /right/col1: track 133.4 -> 0.00 mm
- net /left/row0: track 0.00 -> 104.2 mm
- net /left/row1: track 0.00 -> 103.8 mm
- net /left/row2: track 0.00 -> 103.7 mm
- net /left/col4: track 55.1 -> 0.00 mm
- net Net-(D9-A): track 0.00 -> 38.7 mm
- net /left/col3: track 26.6 -> 0.00 mm
- net /left/vbat: track 22.9 -> 0.00 mm
- net GND: track 22.1 -> 0.00 mm
- net Net-(D11-A): track 0.00 -> 13.6 mm
- net Net-(D51-A): track 13.2 -> 0.00 mm

Commit message: save after kicad cntrl + s
Routing:
- net /left/col4: track 0.00 -> 364.8 mm
- net /left/row4: track 0.00 -> 287.0 mm
- net /left/col5: track 0.00 -> 223.6 mm, vias 0 -> 1
- net /left/col3: track 0.00 -> 218.1 mm
- net /left/row3: track 0.00 -> 201.6 mm, vias 0 -> 2
- net /left/col2: track 0.00 -> 168.3 mm, vias 0 -> 1
- net /left/col1: track 0.00 -> 128.3 mm, vias 0 -> 1
- net /left/col0: track 0.00 -> 122.5 mm, vias 0 -> 1
- net Net-(D35-A): track 0.00 -> 99.3 mm
- net /left/row2: track 103.7 -> 179.3 mm, vias 0 -> 2
- net /left/row1: track 103.8 -> 169.6 mm, vias 0 -> 2
- net Net-(D25-A): track 0.00 -> 61.7 mm
- net Net-(D3-A): track 0.00 -> 58.5 mm
- net GND: track 0.00 -> 57.7 mm, vias 0 -> 1
- net Net-(D23-A): track 0.00 -> 57.3 mm
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
Commit message: save before GND fix
Routing:
- net GND: track 57.7 -> 70.5 mm, vias 1 -> 3
Changed lines of the file:
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@@
+		(net 85)
+	)
+	(segment
+		(start 43.899 26.601)
+		(end 46 24.5)
+		(width 0.2)
+		(layer "F.Cu")
+		(net 85)
+	)
+	(segment
+		(start 41.101 26.601)
+		(end 43.899 26.601)
+		(width 0.2)
+		(layer "F.Cu")
+		(net 85)
+	)
+	(segment
+		(start 50 23.5)
+		(end 50.08 23.42)
+		(width 0.2)
+		(layer "F.Cu")
+		(net 85)
+	)
+	(segment
+		(start 50.08 23.42)
+		(end 52.555 23.42)
+		(width 0.2)
+		(layer "F.Cu")
+		(net 85)
+	)
+	(via
+		(at 46 24.5)
+		(size 0.6)
+		(drill 0.3)
+		(layers "F.Cu" "B.Cu")
 		(net 85)
 	)
@@
 		(drill 0.3)
 		(layers "F.Cu" "B.Cu")
+		(net 85)
+	)
+	(via
+		(at 50 23.5)
+		(size 0.6)
+		(drill 0.3)
+		(layers "F.Cu" "B.Cu")
+		(net 85)
+	)
+	(segment
+		(start 49 24.5)
+		(end 50 23.5)
+		(width 0.2)
+		(layer "B.Cu")
 		(net 85)
 	)
@@
 		(width 0.2)
 		(layer "B.Cu")
+		(net 85)
+	)
+	(segment
+		(start 46 24.5)
+		(end 49 24.5)
+		(width 0.2)
+		(layer "B.Cu")

Commit message: Finalllyyy i fixed my mousebites problem
Parts:
- removed H10, H11, H12, H13, H2, H4, H6, H7, H8, H9: MountingHole, panelization:mouse-bite-5mm-slot
Routing:
- net /right/row3: track 0.00 -> 237.6 mm, vias 0 -> 2
- net /right/col0: track 0.00 -> 222.3 mm
- net /right/row4: track 0.00 -> 193.8 mm, vias 0 -> 2
- net /right/row1: track 0.00 -> 191.9 mm
- net /right/row2: track 0.00 -> 173.8 mm, vias 0 -> 2
- net /right/col1: track 0.00 -> 162.6 mm, vias 0 -> 1
- net /right/row0: track 0.00 -> 142.8 mm
- net /right/col2: track 0.00 -> 134.8 mm, vias 0 -> 1
- net /right/col5: track 0.00 -> 120.1 mm, vias 0 -> 1
- net /right/col3: track 0.00 -> 116.2 mm, vias 0 -> 1
- net /right/col4: track 0.00 -> 105.4 mm, vias 0 -> 1
- net GND: track 70.5 -> 121.2 mm, vias 3 -> 4
- net Net-(D50-A): track 0.00 -> 43.3 mm
- net Net-(D52-A): track 0.00 -> 42.8 mm
- net Net-(D48-A): track 0.00 -> 41.0 mm
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Other:
- board size 251 x 122.9 mm -> 253 x 123 mm

Commit message: save (last commit wasn't with the project fully up-to-date)
Parts:
- added SW61: RotaryEncoder, Rotary_Encoder:RotaryEncoder_Alps_EC11E-Switch_Vertical_H20mm, F.Cu at (61.8, 21.3)
- added SW62: RotaryEncoder, Rotary_Encoder:RotaryEncoder_Alps_EC11E-Switch_Vertical_H20mm, F.Cu at (230.9, 21.3)
Connections:
- U1 pad 17: unconnected-(U1-NFC1-Pad17) -> Net-(U1-NFC1)
- U1 pad 18: unconnected-(U1-NFC2-Pad18) -> Net-(U1-NFC2)
- U1 pad 22: unconnected-(U1-GND-Pad22) -> Net-(SW61-PadC)
- U2 pad 17: unconnected-(U2-NFC1-Pad17) -> Net-(U2-NFC1)
- U2 pad 18: unconnected-(U2-NFC2-Pad18) -> Net-(U2-NFC2)
- U2 pad 22: unconnected-(U2-GND-Pad22) -> Net-(SW62-PadC)
Routing:
- net Net-(U1-NFC1): track 0.00 -> 82.9 mm, vias 0 -> 2
- net Net-(U1-NFC2): track 0.00 -> 71.5 mm, vias 0 -> 2
- net Net-(U2-NFC1): track 0.00 -> 53.3 mm, vias 0 -> 1
- net Net-(U2-NFC2): track 0.00 -> 47.6 mm, vias 0 -> 1
- net Net-(SW62-PadC): track 0.00 -> 36.6 mm, vias 0 -> 1
- net Net-(SW61-PadC): track 0.00 -> 18.3 mm, vias 0 -> 2
- net /left/col1: track 128.3 -> 131.0 mm
Other:
- board size 253 x 123 mm -> 253 x 126.5 mm
