File: bluekeeb-kicad/bluekeeb.kicad_pcb (KiCad board)
At the start: 2 copper layers, 253 x 126.5 mm, 131 parts, among them SW1 SW_Push, SW10 SW_Push, SW11 SW_Push, SW12 SW_Push, SW13 SW_Push, SW14 SW_Push, SW15 SW_Push, SW16 SW_Push, SW17 SW_Push, SW18 SW_Push, SW19 SW_Push, SW2 SW_Push, SW20 SW_Push, SW21 SW_Push, SW22 SW_Push, SW23 SW_Push, SW24 SW_Push, SW25 SW_Push, SW26 SW_Push, SW27 SW_Push, SW28 SW_Push, SW29 SW_Push, SW3 SW_Push, SW30 SW_Push, SW31 SW_Push, SW32 SW_Push, SW33 SW_Push, SW34 SW_Push, SW35 SW_Push, SW36 SW_Push, SW37 SW_Push, SW38 SW_Push, SW39 SW_Push, SW4 SW_Push, SW40 SW_Push, SW41 SW_Push, SW42 SW_Push, SW43 SW_Push, SW44 SW_Push, SW45 SW_Push, SW46 SW_Push, SW47 SW_Push, SW48 SW_Push, SW49 SW_Push, SW5 SW_Push, SW50 SW_Push, SW51 SW_Push, SW52 SW_Push, SW53 SW_Push, SW54 SW_Push, SW55 SW_Push, SW56 SW_Push, SW57 SW_Push, SW58 SW_Push, SW59 SW_Push, SW6 SW_Push, SW60 SW_Push, SW61 RotaryEncoder, SW62 RotaryEncoder, SW7 SW_Push, SW8 SW_Push, SW9 SW_Push, U1 XIAO-nRF52840-SMD, U2 XIAO-nRF52840-SMD

Commit message: added some mounting holes, and i moved the testpoints to a different location.
Parts:
- added H14: MountingHole, MountingHole:MountingHole_2.2mm_M2, F.Cu at (205.0, 132.5)
- added H15: MountingHole, MountingHole:MountingHole_2.2mm_M2, F.Cu at (102.5, 132.5)
- added H16: MountingHole, MountingHole:MountingHole_2.2mm_M2, F.Cu at (226.0, 18.5)
- added H17: MountingHole, MountingHole:MountingHole_2.2mm_M2, F.Cu at (82.5, 19.5)
- added H18: MountingHole, MountingHole:MountingHole_2.2mm_M2, F.Cu at (275.5, 89.0)
- added H19: MountingHole, MountingHole:MountingHole_2.2mm_M2, F.Cu at (30.5, 100.5)
- moved TP3 55.5 mm to (82.5, 26.0)
- moved TP4 54.6 mm to (226.0, 24.5)
- moved TP1 51.3 mm to (82.5, 31.0)
- moved TP2 50.1 mm to (226.0, 30.5)
Routing:
- net /left/vbat: track 18.5 -> 101.2 mm, vias 1 -> 7
- net GND: track 121.2 -> 189.1 mm, vias 4 -> 7
- net /right/vbat: track 24.5 -> 41.2 mm, vias 0 -> 1
- net /left/col2: track 168.3 -> 170.2 mm
Other:
- outline, holes or cut-outs redrawn
